Commit message: v2.0

File: src/sixrobot_description/urdf/sixrobot.urdf (robot description, URDF)
Before this commit: robot sixrobot, 7 links, 6 joints
Links:
- link Link1: mass 2.9711 -> 3.1834; geometry collision mesh filename=package://sixrobot/meshes/Link1.stl; visual mesh filename=package://sixrobot/meshes/Link1.stl
- link Link2: mass 1.2043 -> 2.1027; geometry collision mesh filename=package://sixrobot/meshes/Link2.stl; visual mesh filename=package://sixrobot/meshes/Link2.stl
- link Link3: mass 0.79833 -> 1.9613; geometry collision mesh filename=package://sixrobot/meshes/Link3.stl; visual mesh filename=package://sixrobot/meshes/Link3.stl
- link Link4: mass 0.77257 -> 1.7626; geometry collision mesh filename=package://sixrobot/meshes/Link4.stl; visual mesh filename=package://sixrobot/meshes/Link4.stl
- link Link5: mass 0.7621 -> 1.9415; geometry collision mesh filename=package://sixrobot/meshes/Link5.stl; visual mesh filename=package://sixrobot/meshes/Link5.stl
- link Link6: mass 0.28753 -> 0.049116; geometry collision mesh filename=package://sixrobot/meshes/Link6.stl; visual mesh filename=package://sixrobot/meshes/Link6.stl
- link base_link: mass 4.0022 -> 3.0395; geometry collision mesh filename=package://sixrobot/meshes/base_link.stl; visual mesh filename=package://sixrobot/meshes/base_link.stl
Joints:
- joint joint1: limit lower=-1.57 upper=1.57 effort=0 velocity=0 -> lower=-1.5708 upper=1.5708 effort=0 velocity=0; origin xyz=0.14553 0.082167 0.0937 rpy=1.5708 1.2811E-08 1.5708 -> xyz=-0.0088055 -0.022514 0.09434 rpy=1.5708 5.6825E-17 1.1891
- joint joint2: axis 0 0 1 -> 0 0 -1; limit lower=0.296 upper=3.768 effort=0 velocity=0 -> lower=-1.5708 upper=1.5708 effort=0 velocity=0; origin xyz=-0.053834 0.12 0 rpy=-4.996E-14 -1.6098E-13 -2.8449 -> xyz=-0.005 0.1 0 rpy=3.1416 -1.1269E-15 1.5708
- joint joint3: axis 0 0 1 -> 0 0 -1; limit lower=-3.14 upper=0 effort=0 velocity=0 -> lower=-1.5708 upper=1.5708 effort=0 velocity=0; origin xyz=-0.19 0 0 rpy=-4.4409E-14 -1.4433E-13 -3.1416 -> xyz=0.205 0 0 rpy=-1.1102E-16 1.6099E-16 3.1416
- joint joint4: axis -1 0 0 -> 0.97722 0.12611 0.17071; origin xyz=0 0.072 0 rpy=-8.3267E-15 1.0547E-13 6.4893E-14 -> xyz=-0.11 0 0 rpy=-0.13967 0.1538 1.4216
- joint joint5: axis 0.083262 0.063107 0.99453 -> 0 0 -1; limit lower=-0.69 upper=1.57 effort=0 velocity=0 -> lower=-1.5708 upper=1.5708 effort=0 velocity=0; origin xyz=-0.182 0 0 rpy=0.06337 -0.083358 -0.060704 -> xyz=0.20277 0.026168 0.035423 rpy=-0.11711 0.17155 -3.0132
- joint joint6: axis 0 0 1 -> -1 0 0; limit lower=-1.5708 upper=1.5708 effort=0 velocity=0 -> (none); origin xyz=-0.046785 -0.001336 0.0040016 rpy=-0.61742 -1.4661 0.64856 -> xyz=-0.13508 0 0.000625 rpy=-1.8616 -2.3315E-15 8.5363E-18; type revolute -> continuous

File: src/sixrobot_description/urdf/urdf/sixrobot_base.urdf (robot description, URDF)
Before this commit: robot sixrobot, 7 links, 6 joints
Links:
- link Link1: mass 2.9711 -> 3.1834
- link Link2: mass 1.2043 -> 2.1027
- link Link3: mass 0.79833 -> 1.9613
- link Link4: mass 0.77257 -> 1.7626
- link Link5: mass 0.7621 -> 1.9415
- link Link6: mass 0.28753 -> 0.049116
- link base_link: mass 4.0022 -> 3.0395
Joints:
- joint joint1: limit lower=-1.57 upper=1.57 effort=0 velocity=0 -> lower=-1.5708 upper=1.5708 effort=0 velocity=0; origin xyz=0.14553 0.082167 0.0937 rpy=1.5708 1.2811E-08 1.5708 -> xyz=-0.0088055 -0.022514 0.09434 rpy=1.5708 5.6825E-17 1.1891
- joint joint2: axis 0 0 1 -> 0 0 -1; limit lower=0.296 upper=3.768 effort=0 velocity=0 -> lower=-1.5708 upper=1.5708 effort=0 velocity=0; origin xyz=-0.053834 0.12 0 rpy=-4.996E-14 -1.6098E-13 -2.8449 -> xyz=-0.005 0.1 0 rpy=3.1416 -1.1269E-15 1.5708
- joint joint3: axis 0 0 1 -> 0 0 -1; limit lower=-3.14 upper=0 effort=0 velocity=0 -> lower=-1.5708 upper=1.5708 effort=0 velocity=0; origin xyz=-0.19 0 0 rpy=-4.4409E-14 -1.4433E-13 -3.1416 -> xyz=0.205 0 0 rpy=-1.1102E-16 1.6099E-16 3.1416
- joint joint4: axis -1 0 0 -> 0.97722 0.12611 0.17071; origin xyz=0 0.072 0 rpy=-8.3267E-15 1.0547E-13 6.4893E-14 -> xyz=-0.11 0 0 rpy=-0.13967 0.1538 1.4216
- joint joint5: axis 0.083262 0.063107 0.99453 -> 0 0 -1; limit lower=-0.69 upper=1.57 effort=0 velocity=0 -> lower=-1.5708 upper=1.5708 effort=0 velocity=0; origin xyz=-0.182 0 0 rpy=0.06337 -0.083358 -0.060704 -> xyz=0.20277 0.026168 0.035423 rpy=-0.11711 0.17155 -3.0132
- joint joint6: axis 0 0 1 -> -1 0 0; limit lower=-1.5708 upper=1.5708 effort=0 velocity=0 -> (none); origin xyz=-0.046785 -0.001336 0.0040016 rpy=-0.61742 -1.4661 0.64856 -> xyz=-0.13508 0 0.000625 rpy=-1.8616 -2.3315E-15 8.5363E-18; type revolute -> continuous

File: src/sixrobot_description/urdf/urdf/sixrobot_with_camera.urdf (robot description, URDF)
Before this commit: robot sixrobot, 8 links, 7 joints
Links:
- link camera_link: geometry visual box size=0.04 0.02 0.02
Joints:
- joint camera_joint: origin xyz=0.17 0 0.10 rpy=0 0 0 -> xyz=0.14555 0 0.10 rpy=0 0 0

File: src/sixrobot_description/urdf/xacro/gazebo/sixrobot_base_gazebo.xacro (robot description, xacro)
@@ -102,23 +102,3 @@
     </actuator>
   </transmission>
-  <!-- controller -->
-  <gazebo>
-      <plugin name="ros_control"
-              filename="libgazebo_ros_control.so">
-          <rosDebugLevel>Debug</rosDebugLevel>
-          <publishTF>true</publishTF>
-          <robotNamespace>/</robotNamespace>
-          <robotSimType>gazebo_ros_control/DefaultRobotHWSim</robotSimType>
-          <publishTf>1</publishTf>
-          <publishJointState>true</publishJointState>
-          <alwaysOn>true</alwaysOn>
-          <updateRate>100.0</updateRate>
-          <legacyMode>true</legacyMode>
-          <broadcastTF>1</broadcastTF>
-          <Torque>30</Torque>
-          <Acceleration>1.8</Acceleration>
-          <commandTopic>cmd_vel</commandTopic>
-          <robotBaseFrame>world</robotBaseFrame>
-      </plugin>
-  </gazebo>
 </robot>

File: src/sixrobot_description/urdf/xacro/gazebo/sixrobot_gazebo.xacro (robot description, xacro)
@@ -1,5 +1,475 @@
-<?xml version="1.0"?>
+<?xml version="1.0" ?>
 <robot name="sixrobot" xmlns:xacro="http://www.ros.org/wiki/xacro">
+  <xacro:arg name="gazebo" default="false"/>
+  <xacro:if value="$(arg gazebo)">
+    <!-- Gazebo Tags -->
     <xacro:include filename="$(find sixrobot_description)/urdf/xacro/gazebo/sixrobot_base_gazebo.xacro" />
-    <sixrobot_base_gazebo/>
+  </xacro:if>
+  <virtual_joint name="world_joint" type="fixed" parent_frame="world_frame" child_link="base_link" />
+  <link name="world"/>
+  <joint name="fixed" type="fixed">
+  <parent link="world"/>
+  <child link="base_link"/>
+  </joint>
+  <link
+    name="base_link">
+    <inertial>
+      <origin
+        xyz="0.14555 0.062586 -0.15713"
+        rpy="0 0 0" />
+      <mass
+        value="4.0022" />
+      <inertia
+        ixx="0.012253"
+        ixy="-2.6729E-06"
+        ixz="2.0656E-06"
+        iyy="0.0093348"
+        iyz="0.0019878"
+        izz="0.003386" />
+    </inertial>
+    <visual>
+      <origin
+        xyz="0 0 0"
+        rpy="0 0 0" />
+      <geometry>
+        <mesh
+          filename="package://sixrobot_description/meshes/base_link.stl" />
+      </geometry>
+      <material name="white"/>
+    </visual>
+    <collision>
+      <origin
+        xyz="0 0 0"
+        rpy="0 0 0" />
+      <geometry>
+        <mesh
+          filename="package://sixrobot_description/meshes/base_link.stl" />
+      </geometry>
+    </collision>
+  </link>
+  <link
+    name="Link1">
+    <inertial>
+      <origin
+        xyz="0.014283 0.062229 -0.0073351"
+        rpy="0 0 0" />
+      <mass
+        value="2.9711" />
+      <inertia
+        ixx="0.0030896"
+        ixy="4.1872E-05"
+        ixz="-0.0003107"
+        iyy="0.004441"
+        iyz="1.6622E-05"
+        izz="0.0027928" />
+    </inertial>
+    <visual>
+      <origin
+        xyz="0 0 0"
+        rpy="0 0 0" />
+      <geometry>
+        <mesh
+          filename="package://sixrobot_description/meshes/Link1.stl" />
+      </geometry>
+      <material name="red"/>
+    </visual>
+    <collision>
+      <origin
+        xyz="0 0 0"
+        rpy="0 0 0" />
+      <geometry>
+        <mesh
+          filename="package://sixrobot_description/meshes/Link1.stl" />
+      </geometry>
+    </collision>
+  </link>
+  <joint
+    name="joint1"
+    type="fixed">
+    <origin
+      xyz="0.14553 0.082167 0.0937"
+      rpy="1.5708 1.2811E-08 1.5708" />
+    <parent
+      link="base_link" />
+    <child
+      link="Link1" />
+    <axis
+      xyz="0 1 0" />
+    <limit
+      lower="-1.57"
+      upper="1.57"
+      effort="0"
+      velocity="0" />
+  </joint>
+  <link
+    name="Link2">
+    <inertial>
+      <origin
+        xyz="-0.081903 -6.2825E-05 -0.0062784"
+        rpy="0 0 0" />
+      <mass
+        value="1.2043" />
+      <inertia
+        ixx="0.0012825"
+        ixy="-4.0552E-06"
+        ixz="-0.0004638"
+        iyy="0.0034706"
+        iyz="-3.3631E-06"
+        izz="0.0022087" />
+    </inertial>
+    <visual>
+      <origin
+        xyz="0 0 0"
+        rpy="0 0 0" />
+      <geometry>
+        <mesh
+          filename="package://sixrobot_description/meshes/Link2.stl" />
+      </geometry>
+      <material name="green"/>
+    </visual>
+    <collision>
+      <origin
+        xyz="0 0 0"
+        rpy="0 0 0" />
+      <geometry>
+        <mesh
+          filename="package://sixrobot_description/meshes/Link2.stl" />
+      </geometry>
+    </collision>
+  </link>
+  <joint
+    name="joint2"
+    type="fixed">
+    <origin
+      xyz="-0.053834 0.12 0"
+      rpy="-4.996E-14 -1.6098E-13 -2.8449" />
+    <parent
+      link="Link1" />
+    <child
+      link="Link2" />
+    <axis
+      xyz="0 0 1" />
+    <limit
+      lower="0.296"
+      upper="3.768"
+      effort="0"
+      velocity="0" />
+  </joint>
+  <link
+    name="Link3">
+    <inertial>
+      <origin
+        xyz="-0.0030891 0.053464 0.0015565"
+        rpy="0 0 0" />
+      <mass
+        value="0.79833" />
+      <inertia
+        ixx="0.0019731"
+        ixy="0.00011484"
+        ixz="-4.1195E-06"
+        iyy="0.00037597"
+        iyz="6.6446E-05"
+        izz="0.0019652" />
+    </inertial>
+    <visual>
+      <origin
+        xyz="0 0 0"
+        rpy="0 0 0" />
+      <geometry>
+        <mesh
+          filename="package://sixrobot_description/meshes/Link3.stl" />
+      </geometry>
+      <material name="blue"/>
+    </visual>
+    <collision>
+      <origin
+        xyz="0 0 0"
+        rpy="0 0 0" />
+      <geometry>
+        <mesh
+          filename="package://sixrobot_description/meshes/Link3.stl" />
+      </geometry>
+    </collision>
+  </link>
+  <joint
+    name="joint3"
+    type="fixed">
+    <origin
+      xyz="-0.19 0 0"
+      rpy="-4.4409E-14 -1.4433E-13 -3.1416" />
+    <parent
+      link="Link2" />
+    <child
+      link="Link3" />
+    <axis
+      xyz="0 0 1" />
+    <limit
+      lower="-3.14"
+      upper="0"
+      effort="0"
+      velocity="0" />
+  </joint>
+  <link
+    name="Link4">
+    <inertial>
+      <origin
+        xyz="-0.10243 0.00012682 -0.0034682"
+        rpy="0 0 0" />
+      <mass
+        value="0.77257" />
+      <inertia
+        ixx="0.00045081"
+        ixy="-4.7414E-06"
+        ixz="-1.86E-05"
+        iyy="0.0019073"
+        iyz="-8.0337E-08"
+        izz="0.0014729" />
+    </inertial>
+    <visual>
+      <origin
+        xyz="0 0 0"
+        rpy="0 0 0" />
+      <geometry>
+        <mesh
+          filename="package://sixrobot_description/meshes/Link4.stl" />
+      </geometry>
+      <material name="red"/>
+    </visual>
+    <collision>
+      <origin
+        xyz="0 0 0"
+        rpy="0 0 0" />
+      <geometry>
+        <mesh
+          filename="package://sixrobot_description/meshes/Link4.stl" />
+      </geometry>
+    </collision>
+  </link>
+  <joint
+    name="joint4"
+    type="fixed">
+    <origin
+      xyz="0 0.072 0"
+      rpy="-8.3267E-15 1.0547E-13 6.4893E-14" />
+    <parent
+      link="Link3" />
+    <child
+      link="Link4" />
+    <axis
+      xyz="-1 0 0" />
+    <limit
+      lower="-1.5708"
+      upper="1.5708"
+      effort="0"
+      velocity="0" />
+  </joint>
+  <link
+    name="Link5">
+    <inertial>
+      <origin
+        xyz="-0.03177 0.012539 -0.0082766"
+        rpy="0 0 0" />
+      <mass
+        value="0.7621" />
+      <inertia
+        ixx="0.00088662"
+        ixy="0.00027254"
+        ixz="0.00023505"
+        iyy="0.0011014"
+        iyz="-0.00012409"
+        izz="0.0010153" />
+    </inertial>
+    <visual>
+      <origin
+        xyz="0 0 0"
+        rpy="0 0 0" />
+      <geometry>
+        <mesh
+          filename="package://sixrobot_description/meshes/Link5.stl" />
+      </geometry>
+      <material name="green"/>
+    </visual>
+    <collision>
+      <origin
+        xyz="0 0 0"
+        rpy="0 0 0" />
+      <geometry>
+        <mesh
+          filename="package://sixrobot_description/meshes/Link5.stl" />
+      </geometry>
+    </collision>
+  </link>
+  <joint
+    name="joint5"
+    type="fixed">
+    <origin
+      xyz="-0.182 0 0"
+      rpy="0.06337 -0.083358 -0.060704" />
+    <parent
+      link="Link4" />
+    <child
+      link="Link5" />
+    <axis
+      xyz="0.083262 0.063107 0.99453" />
+    <limit
+      lower="-0.69"
+      upper="1.57"
+      effort="0"
+      velocity="0" />
+  </joint>
+  <link
+    name="Link6">
+    <inertial>
+      <origin
+        xyz="4.8525E-06 -0.00027138 0.054503"
+        rpy="0 0 0" />
+      <mass
+        value="0.28753" />
+      <inertia
+        ixx="5.4771E-05"
+        ixy="2.9237E-08"
+        ixz="4.993E-09"
+        iyy="5.4752E-05"
+        iyz="4.997E-08"
+        izz="3.9349E-06" />
+    </inertial>
+    <visual>
+      <origin
+        xyz="0 0 0"
+        rpy="0 0 0" />
+      <geometry>
+        <mesh
+          filename="package://sixrobot_description/meshes/Link6.stl" />
+      </geometry>
+      <material name="blue"/>
+    </visual>
+    <collision>
+      <origin
+        xyz="0 0 0"
+        rpy="0 0 0" />
+      <geometry>
+        <mesh
+          filename="package://sixrobot_description/meshes/Link6.stl" />
+      </geometry>
+    </collision>
+  </link>
+  <joint
+    name="joint6"
+    type="fixed">
+    <origin
+      xyz="-0.046785 -0.001336 0.0040016"
+      rpy="-0.61742 -1.4661 0.64856" />
+    <parent
+      link="Link5" />
+    <child
+      link="Link6" />
+    <axis
+      xyz="0 0 1" />
+    <limit
+      lower="-1.5708"
+      upper="1.5708"
+      effort="0"
+      velocity="0" />
+  </joint>
+  <!-- ros_control plugin -->
+  <gazebo>
+    <plugin name="ros_control" filename="lib_gazebo_ros_control.so">
+      <robotNamespace>/robot</robotNamespace>
+    </plugin>
+  </gazebo>
+  <!-- Gazebo-Specific Link Properties -->
+  <gazebo reference="world_joint">
+    <selfCollide>true</selfCollide>
+    <material>Gazebo/White</material>
+  </gazebo>
+  <gazebo reference="base_link">
+    <selfCollide>true</selfCollide>
+    <material>Gazebo/White</material>
+  </gazebo>
+  <gazebo reference="Link1">
+    <implicitSpringDamper>1</implicitSpringDamper>
+    <material>Gazebo/Red</material>
+  </gazebo>
+  <gazebo reference="Link2">
+    <implicitSpringDamper>1</implicitSpringDamper>
+    <material>Gazebo/Green</material>
+  </gazebo>
+  <gazebo reference="Link3">
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
File: src/sixrobot_description/urdf/xacro/gazebo/sixrobot_with_camera_gazebo.xacro (robot description, xacro)
@@ -3,10 +3,5 @@
     <xacro:arg name="gazebo" default="false"/>
     <!-- sixrobot Base URDF -->
-    <xacro:include filename="$(find sixrobot_description)/urdf/xacro/gazebo/sixrobot_base_gazebo.xacro">
-        <xacro:arg name="gazebo" value="${gazebo}"/>
-    </xacro:include>
-    <xacro:arg name="gazebo" default="false"/>
-    <!-- sixrobot Base URDF -->
-    <xacro:include filename="$(find sixrobot_description)/urdf/xacro/gazebo/sixrobot_base.urdf.xacro">
+    <xacro:include filename="$(find sixrobot_description)/urdf/xacro/gazebo/sixrobot_gazebo.xacro">
         <xacro:arg name="gazebo" value="${gazebo}"/>
     </xacro:include>
@@ -16,5 +11,5 @@
         <xacro:arg name="gazebo" value="${gazebo}"/>
     </xacro:include>
-    <xacro:property name="camera_offset_x" value="0.17" />
+    <xacro:property name="camera_offset_x" value="0.14555" />
     <xacro:property name="camera_offset_y" value="0" />
     <xacro:property name="camera_offset_z" value="0.10" />
@@ -22,5 +17,5 @@
     <joint name="camera_joint" type="fixed">
         <origin xyz="${camera_offset_x} ${camera_offset_y} ${camera_offset_z}" rpy="0 0 0" />
-        <parent link="world"/>
+        <parent link="base_link"/>
         <child link="camera_link"/>
     </joint>

File: src/sixrobot_description/urdf/xacro/gazebo/sixrobot_with_kinect_gazebo.xacro (robot description, xacro)
@@ -3,10 +3,5 @@
     <xacro:arg name="gazebo" default="false"/>
     <!-- sixrobot Base URDF -->
-    <xacro:include filename="$(find sixrobot_description)/urdf/xacro/gazebo/sixrobot_base_gazebo.xacro">
-        <xacro:arg name="gazebo" value="${gazebo}"/>
-    </xacro:include>
-    <xacro:arg name="gazebo" default="false"/>
-    <!-- sixrobot Base URDF -->
-    <xacro:include filename="$(find sixrobot_description)/urdf/xacro/gazebo/sixrobot_base.urdf.xacro">
+    <xacro:include filename="$(find sixrobot_description)/urdf/xacro/gazebo/sixrobot_gazebo.xacro">
         <xacro:arg name="gazebo" value="${gazebo}"/>
     </xacro:include>
@@ -16,5 +11,5 @@
         <xacro:arg name="gazebo" value="${gazebo}"/>
     </xacro:include>
-    <xacro:property name="kinect_offset_x" value="0.7" />
+    <xacro:property name="kinect_offset_x" value="0.14555" />
     <xacro:property name="kinect_offset_y" value="0" />
     <xacro:property name="kinect_offset_z" value="0.11" />

File: src/sixrobot_description/urdf/xacro/gazebo/sixrobot_with_laser_gazebo.xacro (robot description, xacro)
@@ -3,10 +3,5 @@
     <xacro:arg name="gazebo" default="false"/>
     <!-- sixrobot Base URDF -->
-    <xacro:include filename="$(find sixrobot_description)/urdf/xacro/gazebo/sixrobot_base_gazebo.xacro">
-        <xacro:arg name="gazebo" value="${gazebo}"/>
-    </xacro:include>
-    <xacro:arg name="gazebo" default="false"/>
-    <!-- sixrobot Base URDF -->
-    <xacro:include filename="$(find sixrobot_description)/urdf/xacro/gazebo/sixrobot_base.urdf.xacro">
+    <xacro:include filename="$(find sixrobot_description)/urdf/xacro/gazebo/sixrobot_gazebo.xacro">
         <xacro:arg name="gazebo" value="${gazebo}"/>
     </xacro:include>
@@ -16,5 +11,5 @@
         <xacro:arg name="gazebo" value="${gazebo}"/>
     </xacro:include>
-    <xacro:property name="lidar_offset_x" value="0" />
+    <xacro:property name="lidar_offset_x" value="0.14555" />
     <xacro:property name="lidar_offset_y" value="0" />
     <xacro:property name="lidar_offset_z" value="0.105" />

File: src/sixrobot_description/urdf/xacro/sensors/camera.xacro (robot description, xacro)
@@ -6,5 +6,5 @@
                 <origin xyz=" 0 0 0 " rpy="0 0 0" />
                 <geometry>
-                    <box size="0.01 0.04 0.04" />
+                    <box size="0.04 0.02 0.02" />
                 </geometry>
                 <material name="red"/>

File: src/sixrobot_description/urdf/xacro/sensors/camera_gazebo.xacro (robot description, xacro)
@@ -6,25 +6,29 @@
             <inertial>
                 <mass value="0.1" />
-                <origin xyz="0 0 0" />
-                <inertia ixx="0.01" ixy="0.0" ixz="0.0"
-                         iyy="0.01" iyz="0.0"
-                         izz="0.01" />
+                <origin xyz="0 0 0.054503"
+                        rpy="0 0 0" />
+                <inertia ixx="5.4771E-05"
+                         ixy="2.9237E-08"
+                         ixz="4.993E-09"
+                         iyy="5.4752E-05"
+                         iyz="4.997E-08"
+                         izz="3.9349E-06" />
             </inertial>
             <visual>
                 <origin xyz=" 0 0 0 " rpy="0 0 0" />
                 <geometry>
-                    <box size="0.01 0.04 0.04" />
+                    <box size="0.04 0.02 0.02" />
                 </geometry>
-                <material name="red"/>
+                <material name="black"/>
             </visual>
             <collision>
                 <origin xyz="0.0 0.0 0.0" rpy="0 0 0" />
                 <geometry>
-                    <box size="0.01 0.04 0.04" />
+                    <box size="0.04 0.02 0.02" />
                 </geometry>
             </collision>
         </link>
         <gazebo reference="${prefix}_link">
-            <material>Gazebo/Red</material>
+            <material>Gazebo/Black</material>
         </gazebo>
         <gazebo reference="${prefix}_link">

File: src/sixrobot_description/urdf/xacro/sensors/kinect.xacro (robot description, xacro)
@@ -2,7 +2,7 @@
 <robot xmlns:xacro="http://www.ros.org/wiki/xacro" name="kinect_camera">
     <xacro:macro name="kinect_camera" params="prefix:=camera">
-    <property name="PI" value="3.14159265" />
+    <xacro:property name="PI" value="3.14159265" />
         <link name="${prefix}_link">
-            <origin xyz="4.8525E-06 -0.00027138 0.054503"
+            <origin xyz="0 0 0"
         rpy="0 0 0"/>
             <visual>
@@ -14,6 +14,6 @@
         </link>
         <joint name="${prefix}_optical_joint" type="fixed">
-            <origin xyz="-0.046785 -0.001336 0.0040016"
-      rpy="-0.61742 -1.4661 0.64856"/>
+            <origin xyz="0 0 0"
+      rpy="0 0 0" />
             <parent link="${prefix}_link"/>
             <child link="${prefix}_frame_optical"/>
