Commit message: v2.0

File: src/sixrobot_description/urdf/xacro/sensors/kinect_gazebo.xacro (robot description, xacro)
@@ -2,9 +2,9 @@
 <robot xmlns:xacro="http://www.ros.org/wiki/xacro" name="kinect_camera">
     <xacro:macro name="kinect_camera" params="prefix:=camera">
-    <property name="PI" value="3.14159265" />
+    <xacro:property name="PI" value="3.14159265" />
         <!-- Create kinect reference frame -->
         <!-- Add mesh for kinect -->
         <link name="${prefix}_link">
-            <origin xyz="4.8525E-06 -0.00027138 0.054503"
+            <origin xyz="0 0 0"
         rpy="0 0 0"/>
             <visual>
@@ -13,14 +13,25 @@
                     <mesh filename="package://sixrobot_description/meshes/kinect.dae" />
                 </geometry>
+                <material
+                  name="">
+                  <color
+                    rgba="245 245 245 1" />
+                </material>
             </visual>
             <collision>
-                <geometry>
+               <origin
+                  xyz="0 0 0"
+                  rpy="0 0 0" />
+               <geometry>
                     <box size="0.07 0.3 0.09"/>
                 </geometry>
             </collision>
         </link>
+        <gazebo reference="${prefix}_link">
+            <material>Gazebo/Black</material>
+        </gazebo>
         <joint name="${prefix}_optical_joint" type="fixed">
-            <origin xyz="-0.046785 -0.001336 0.0040016"
-      rpy="-0.61742 -1.4661 0.64856"/>
+            <origin xyz="0 0 0"
+      rpy="0 0 0"/>
             <parent link="${prefix}_link"/>
             <child link="${prefix}_frame_optical"/>

File: src/sixrobot_description/urdf/xacro/sensors/lidar.xacro (robot description, xacro)
@@ -6,5 +6,5 @@
 				<origin xyz=" 0 0 0 " rpy="0 0 0" />
 				<geometry>
-					<cylinder length="0.05" radius="0.05"/>
+					<cylinder length="0.02" radius="0.01"/>
 				</geometry>
 				<material name="black"/>

File: src/sixrobot_description/urdf/xacro/sensors/lidar_gazebo.xacro (robot description, xacro)
@@ -14,5 +14,5 @@
                 <origin xyz=" 0 0 0 " rpy="0 0 0" />
                 <geometry>
-                    <cylinder length="0.05" radius="0.05"/>
+                    <cylinder length="0.02" radius="0.01"/>
                 </geometry>
                 <material name="black"/>
@@ -21,5 +21,5 @@
                 <origin xyz="0.0 0.0 0.0" rpy="0 0 0" />
                 <geometry>
-                    <cylinder length="0.06" radius="0.05"/>
+                    <cylinder length="0.02" radius="0.01"/>
                 </geometry>
             </collision>

Commit message: v2.0

File: src/sixrobot_description/urdf/sixrobot.urdf (robot description, URDF)
Before this commit: robot sixrobot, 7 links, 6 joints
Links:
- link Link1: mass 3.1834 -> 0.00001; geometry collision mesh filename=package://sixrobot_description/meshes/Link1.stl; visual mesh filename=package://sixrobot_description/meshes/Link1.stl
- link Link2: mass 2.1027 -> 0.00001; geometry collision mesh filename=package://sixrobot_description/meshes/Link2.stl; visual mesh filename=package://sixrobot_description/meshes/Link2.stl
- link Link3: mass 1.9613 -> 0.00001; geometry collision mesh filename=package://sixrobot_description/meshes/Link3.stl; visual mesh filename=package://sixrobot_description/meshes/Link3.stl
- link Link4: mass 1.7626 -> 0.00001; geometry collision mesh filename=package://sixrobot_description/meshes/Link4.stl; visual mesh filename=package://sixrobot_description/meshes/Link4.stl
- link Link5: mass 1.9415 -> 0.00001; geometry collision mesh filename=package://sixrobot_description/meshes/Link5.stl; visual mesh filename=package://sixrobot_description/meshes/Link5.stl
- link Link6: mass 0.049116 -> 0.00001; geometry collision mesh filename=package://sixrobot_description/meshes/Link6.stl; visual mesh filename=package://sixrobot_description/meshes/Link6.stl
- link base_link: mass 3.0395 -> 0.00001; geometry collision mesh filename=package://sixrobot_description/meshes/base_link.stl; visual mesh filename=package://sixrobot_description/meshes/base_link.stl
Joints:
- joint joint1: limit lower=-1.5708 upper=1.5708 effort=0 velocity=0 -> lower=-1.5708 upper=1.5708 effort=100 velocity=1; origin xyz=-0.0088055 -0.022514 0.09434 rpy=1.5708 5.6825E-17 1.1891 -> xyz=0.00021336 -0.024174 0.09434 rpy=1.5708 6.123E-17 1.5708
- joint joint2: limit lower=-1.5708 upper=1.5708 effort=0 velocity=0 -> lower=-1.5708 upper=1.5708 effort=100 velocity=1; origin xyz=-0.005 0.1 0 rpy=3.1416 -1.1269E-15 1.5708 -> xyz=-0.005 0.1 0 rpy=3.1416 -5.0415E-16 1.5708
- joint joint3: limit lower=-1.5708 upper=1.5708 effort=0 velocity=0 -> lower=-1.5708 upper=1.5708 effort=100 velocity=1; origin xyz=0.205 0 0 rpy=-1.1102E-16 1.6099E-16 3.1416 -> xyz=0.205 0 0 rpy=2.2226E-16 1.2197E-16 3.1416
- joint joint4: limit lower=-1.5708 upper=1.5708 effort=0 velocity=0 -> lower=-1.5708 upper=1.5708 effort=100 velocity=1; origin xyz=-0.11 0 0 rpy=-0.13967 0.1538 1.4216 -> xyz=-0.11 0.0057828 0 rpy=-0.13967 0.1538 1.4216
- joint joint5: limit lower=-1.5708 upper=1.5708 effort=0 velocity=0 -> lower=-1.5708 upper=1.5708 effort=100 velocity=1; origin xyz=0.20277 0.026168 0.035423 rpy=-0.11711 0.17155 -3.0132 -> xyz=0.19712 0.025439 0.034436 rpy=-0.11711 0.17155 -3.0132
- joint joint6: origin xyz=-0.13508 0 0.000625 rpy=-1.8616 -2.3315E-15 8.5363E-18 -> xyz=-0.13059 0 0.000625 rpy=-1.8616 -5.7439E-17 1.638E-17

File: src/sixrobot_description/urdf/urdf/sixrobot_base.urdf (robot description, URDF)
Before this commit: robot sixrobot, 7 links, 6 joints
Links:
- link Link1: mass 3.1834 -> 0.001
- link Link2: mass 2.1027 -> 0.001
- link Link3: mass 1.9613 -> 0.001
- link Link4: mass 1.7626 -> 0.001
- link Link5: mass 1.9415 -> 0.001
- link Link6: mass 0.049116 -> 0.001
- link base_link: mass 3.0395 -> 0.001

File: src/sixrobot_description/urdf/urdf/sixrobot_with_camera.urdf (robot description, URDF)
Before this commit: robot sixrobot, 8 links, 7 joints
Links:
- removed link camera_link
- link Link1: mass 2.9711 -> 0.00001
- link Link2: mass 1.2043 -> 0.00001
- link Link3: mass 0.79833 -> 0.00001
- link Link4: mass 0.77257 -> 0.00001
- link Link5: mass 0.7621 -> 0.00001
- link Link6: mass 0.28753 -> 0.00001
- link base_link: mass 4.0022 -> 0.00001
Joints:
- removed joint camera_joint
- joint joint1: limit lower=-1.57 upper=1.57 effort=0 velocity=0 -> lower=-1.5708 upper=1.5708 effort=0 velocity=0; origin xyz=0.14553 0.082167 0.0937 rpy=1.5708 1.2811E-08 1.5708 -> xyz=-0.0088055 -0.022514 0.09434 rpy=1.5708 5.6825E-17 1.1891
- joint joint2: axis 0 0 1 -> 0 0 -1; limit lower=0.296 upper=3.768 effort=0 velocity=0 -> lower=-1.5708 upper=1.5708 effort=0 velocity=0; origin xyz=-0.053834 0.12 0 rpy=-4.996E-14 -1.6098E-13 -2.8449 -> xyz=-0.005 0.1 0 rpy=3.1416 -1.1269E-15 1.5708
- joint joint3: axis 0 0 1 -> 0 0 -1; limit lower=-3.14 upper=0 effort=0 velocity=0 -> lower=-1.5708 upper=1.5708 effort=0 velocity=0; origin xyz=-0.19 0 0 rpy=-4.4409E-14 -1.4433E-13 -3.1416 -> xyz=0.205 0 0 rpy=-1.1102E-16 1.6099E-16 3.1416
- joint joint4: axis -1 0 0 -> 0.97722 0.12611 0.17071; origin xyz=0 0.072 0 rpy=-8.3267E-15 1.0547E-13 6.4893E-14 -> xyz=-0.11 0 0 rpy=-0.13967 0.1538 1.4216
- joint joint5: axis 0.083262 0.063107 0.99453 -> 0 0 -1; limit lower=-0.69 upper=1.57 effort=0 velocity=0 -> lower=-1.5708 upper=1.5708 effort=0 velocity=0; origin xyz=-0.182 0 0 rpy=0.06337 -0.083358 -0.060704 -> xyz=0.20277 0.026168 0.035423 rpy=-0.11711 0.17155 -3.0132
- joint joint6: axis 0 0 1 -> -1 0 0; limit lower=-1.5708 upper=1.5708 effort=0 velocity=0 -> (none); origin xyz=-0.046785 -0.001336 0.0040016 rpy=-0.61742 -1.4661 0.64856 -> xyz=-0.13508 0 0.000625 rpy=-1.8616 -2.3315E-15 8.5363E-18; type revolute -> continuous

File: src/sixrobot_description/urdf/urdf/sixrobot_with_kinect.urdf (robot description, URDF)
Before this commit: robot sixrobot, 8 links, 7 joints
Links:
- removed link kinect_link
- link Link1: mass 2.9711 -> 0.00001
- link Link2: mass 1.2043 -> 0.00001
- link Link3: mass 0.79833 -> 0.00001
- link Link4: mass 0.77257 -> 0.00001
- link Link5: mass 0.7621 -> 0.00001
- link Link6: mass 0.28753 -> 0.00001
- link base_link: mass 4.0022 -> 0.00001
Joints:
- removed joint kinect_joint
- joint joint1: limit lower=-1.57 upper=1.57 effort=0 velocity=0 -> lower=-1.5708 upper=1.5708 effort=0 velocity=0; origin xyz=0.14553 0.082167 0.0937 rpy=1.5708 1.2811E-08 1.5708 -> xyz=-0.0088055 -0.022514 0.09434 rpy=1.5708 5.6825E-17 1.1891
- joint joint2: axis 0 0 1 -> 0 0 -1; limit lower=0.296 upper=3.768 effort=0 velocity=0 -> lower=-1.5708 upper=1.5708 effort=0 velocity=0; origin xyz=-0.053834 0.12 0 rpy=-4.996E-14 -1.6098E-13 -2.8449 -> xyz=-0.005 0.1 0 rpy=3.1416 -1.1269E-15 1.5708
- joint joint3: axis 0 0 1 -> 0 0 -1; limit lower=-3.14 upper=0 effort=0 velocity=0 -> lower=-1.5708 upper=1.5708 effort=0 velocity=0; origin xyz=-0.19 0 0 rpy=-4.4409E-14 -1.4433E-13 -3.1416 -> xyz=0.205 0 0 rpy=-1.1102E-16 1.6099E-16 3.1416
- joint joint4: axis -1 0 0 -> 0.97722 0.12611 0.17071; origin xyz=0 0.072 0 rpy=-8.3267E-15 1.0547E-13 6.4893E-14 -> xyz=-0.11 0 0 rpy=-0.13967 0.1538 1.4216
- joint joint5: axis 0.083262 0.063107 0.99453 -> 0 0 -1; limit lower=-0.69 upper=1.57 effort=0 velocity=0 -> lower=-1.5708 upper=1.5708 effort=0 velocity=0; origin xyz=-0.182 0 0 rpy=0.06337 -0.083358 -0.060704 -> xyz=0.20277 0.026168 0.035423 rpy=-0.11711 0.17155 -3.0132
- joint joint6: axis 0 0 1 -> -1 0 0; limit lower=-1.5708 upper=1.5708 effort=0 velocity=0 -> (none); origin xyz=-0.046785 -0.001336 0.0040016 rpy=-0.61742 -1.4661 0.64856 -> xyz=-0.13508 0 0.000625 rpy=-1.8616 -2.3315E-15 8.5363E-18; type revolute -> continuous

File: src/sixrobot_description/urdf/urdf/sixrobot_with_laser.urdf (robot description, URDF)
Before this commit: robot sixrobot, 8 links, 7 joints
Links:
- removed link laser_link
- link Link1: mass 2.9711 -> 0.00001
- link Link2: mass 1.2043 -> 0.00001
- link Link3: mass 0.79833 -> 0.00001
- link Link4: mass 0.77257 -> 0.00001
- link Link5: mass 0.7621 -> 0.00001
- link Link6: mass 0.28753 -> 0.00001
- link base_link: mass 4.0022 -> 0.00001
Joints:
- removed joint laser_joint
- joint joint1: limit lower=-1.57 upper=1.57 effort=0 velocity=0 -> lower=-1.5708 upper=1.5708 effort=0 velocity=0; origin xyz=0.14553 0.082167 0.0937 rpy=1.5708 1.2811E-08 1.5708 -> xyz=-0.0088055 -0.022514 0.09434 rpy=1.5708 5.6825E-17 1.1891
- joint joint2: axis 0 0 1 -> 0 0 -1; limit lower=0.296 upper=3.768 effort=0 velocity=0 -> lower=-1.5708 upper=1.5708 effort=0 velocity=0; origin xyz=-0.053834 0.12 0 rpy=-4.996E-14 -1.6098E-13 -2.8449 -> xyz=-0.005 0.1 0 rpy=3.1416 -1.1269E-15 1.5708
- joint joint3: axis 0 0 1 -> 0 0 -1; limit lower=-3.14 upper=0 effort=0 velocity=0 -> lower=-1.5708 upper=1.5708 effort=0 velocity=0; origin xyz=-0.19 0 0 rpy=-4.4409E-14 -1.4433E-13 -3.1416 -> xyz=0.205 0 0 rpy=-1.1102E-16 1.6099E-16 3.1416
- joint joint4: axis -1 0 0 -> 0.97722 0.12611 0.17071; origin xyz=0 0.072 0 rpy=-8.3267E-15 1.0547E-13 6.4893E-14 -> xyz=-0.11 0 0 rpy=-0.13967 0.1538 1.4216
- joint joint5: axis 0.083262 0.063107 0.99453 -> 0 0 -1; limit lower=-0.69 upper=1.57 effort=0 velocity=0 -> lower=-1.5708 upper=1.5708 effort=0 velocity=0; origin xyz=-0.182 0 0 rpy=0.06337 -0.083358 -0.060704 -> xyz=0.20277 0.026168 0.035423 rpy=-0.11711 0.17155 -3.0132
- joint joint6: axis 0 0 1 -> -1 0 0; limit lower=-1.5708 upper=1.5708 effort=0 velocity=0 -> (none); origin xyz=-0.046785 -0.001336 0.0040016 rpy=-0.61742 -1.4661 0.64856 -> xyz=-0.13508 0 0.000625 rpy=-1.8616 -2.3315E-15 8.5363E-18; type revolute -> continuous

File: src/sixrobot_description/urdf/xacro/gazebo/sixrobot_base.urdf.xacro (robot description, xacro)
@@ -19,5 +19,5 @@
         rpy="0 0 0" />
       <mass
-        value="3.0395" />
+        value="0.001" />
       <inertia
         ixx="0.0025797"
@@ -59,5 +59,5 @@
         rpy="0 0 0" />
       <mass
-        value="3.1834" />
+        value="0.001" />
       <inertia
         ixx="0.0066967"
@@ -117,5 +117,5 @@
         rpy="0 0 0" />
       <mass
-        value="2.1027" />
+        value="0.001" />
       <inertia
         ixx="0.0029075"
@@ -175,5 +175,5 @@
         rpy="0 0 0" />
       <mass
-        value="1.9613" />
+        value="0.001" />
       <inertia
         ixx="0.0019119"
@@ -233,5 +233,5 @@
         rpy="0 0 0" />
       <mass
-        value="1.7626" />
+        value="0.001" />
       <inertia
         ixx="0.00091529"
@@ -291,5 +291,5 @@
         rpy="0 0 0" />
       <mass
-        value="1.9415" />
+        value="0.001" />
       <inertia
         ixx="0.0015409"
@@ -349,5 +349,5 @@
         rpy="0 0 0" />
       <mass
-        value="0.049116" />
+        value="0.001" />
       <inertia
         ixx="6.9904E-08"

File: src/sixrobot_description/urdf/xacro/gazebo/sixrobot_base_gazebo.xacro (robot description, xacro)
@@ -3,6 +3,8 @@
   <!-- ros_control plugin -->
   <gazebo>
-    <plugin name="ros_control" filename="lib_gazebo_ros_control.so">
-      <robotNamespace>/robot</robotNamespace>
+    <plugin name="gazebo_ros_control" filename="libgazebo_ros_control.so">
+      <robotNamespace>/sixrobot</robotNamespace>
+      <robotSimType>gazebo_ros_control/DefaultRobotHWSim</robotSimType>
+      <legacyModeNS>true</legacyModeNS>
     </plugin>
   </gazebo>
@@ -40,65 +42,22 @@
     <material>Gazebo/Blue</material>
   </gazebo>
-  <!-- Transmissions -->
-  <!-- Arm -->
-  <transmission name="tran1">
-    <type>transmission_interface/SimpleTransmission</type>
-    <joint name="joint1">
-      <hardwareInterface>EffortJointInterface</hardwareInterface>
-    </joint>
-    <actuator name="motor1">
-      <hardwareInterface>EffortJointInterface</hardwareInterface>
-      <mechanicalReduction>1</mechanicalReduction>
-    </actuator>
-  </transmission>
-  <transmission name="tran2">
-    <type>transmission_interface/SimpleTransmission</type>
-    <joint name="joint2">
-      <hardwareInterface>EffortJointInterface</hardwareInterface>
-    </joint>
-    <actuator name="motor2">
-      <hardwareInterface>EffortJointInterface</hardwareInterface>
-      <mechanicalReduction>1</mechanicalReduction>
-    </actuator>
-  </transmission>
-  <transmission name="tran3">
-    <type>transmission_interface/SimpleTransmission</type>
-    <joint name="joint3">
-      <hardwareInterface>EffortJointInterface</hardwareInterface>
-    </joint>
-    <actuator name="motor3">
-      <hardwareInterface>EffortJointInterface</hardwareInterface>
-      <mechanicalReduction>1</mechanicalReduction>
-    </actuator>
-  </transmission>
-  <transmission name="tran4">
-    <type>transmission_interface/SimpleTransmission</type>
-    <joint name="joint4">
-      <hardwareInterface>EffortJointInterface</hardwareInterface>
-    </joint>
-    <actuator name="motor4">
-      <hardwareInterface>EffortJointInterface</hardwareInterface>
-      <mechanicalReduction>1</mechanicalReduction>
-    </actuator>
-  </transmission>
-  <transmission name="tran5">
-    <type>transmission_interface/SimpleTransmission</type>
-    <joint name="joint5">
-      <hardwareInterface>EffortJointInterface</hardwareInterface>
-    </joint>
-    <actuator name="motor5">
-      <hardwareInterface>EffortJointInterface</hardwareInterface>
-      <mechanicalReduction>1</mechanicalReduction>
-    </actuator>
-  </transmission>
-  <transmission name="tran6">
-    <type>transmission_interface/SimpleTransmission</type>
-    <joint name="joint6">
-      <hardwareInterface>EffortJointInterface</hardwareInterface>
-    </joint>
-    <actuator name="motor6">
-      <hardwareInterface>EffortJointInterface</hardwareInterface>
-      <mechanicalReduction>1</mechanicalReduction>
-    </actuator>
-  </transmission>
+  <!-- Transmissions for ROS Control -->
+  <xacro:macro name="transmission_block" params="joint_name">
+    <transmission name="tran1">
+      <type>transmission_interface/SimpleTransmission</type>
+      <joint name="${joint_name}">
+        <hardwareInterface>hardware_interface/PositionJointInterface</hardwareInterface>
+      </joint>
+      <actuator name="motor1">
+        <hardwareInterface>hardware_interface/PositionJointInterface</hardwareInterface>
+        <mechanicalReduction>1</mechanicalReduction>
+      </actuator>
+    </transmission>
+  </xacro:macro>
+  <xacro:transmission_block joint_name="joint1"/>
+  <xacro:transmission_block joint_name="joint2"/>
+  <xacro:transmission_block joint_name="joint3"/>
+  <xacro:transmission_block joint_name="joint4"/>
+  <xacro:transmission_block joint_name="joint5"/>
+  <xacro:transmission_block joint_name="joint6"/>
 </robot>

File: src/sixrobot_description/urdf/xacro/gazebo/sixrobot_gazebo.xacro (robot description, xacro)
@@ -19,5 +19,5 @@
         rpy="0 0 0" />
       <mass
-        value="3.0395" />
+        value="0.001" />
       <inertia
         ixx="0.0025797"
@@ -59,5 +59,5 @@
         rpy="0 0 0" />
       <mass
-        value="3.1834" />
+        value="0.001" />
       <inertia
         ixx="0.0066967"
@@ -117,5 +117,5 @@
         rpy="0 0 0" />
       <mass
-        value="2.1027" />
+        value="0.001" />
       <inertia
         ixx="0.0029075"
@@ -175,5 +175,5 @@
         rpy="0 0 0" />
       <mass
-        value="1.9613" />
+        value="0.001" />
       <inertia
         ixx="0.0019119"
@@ -233,5 +233,5 @@
         rpy="0 0 0" />
       <mass
-        value="1.7626" />
+        value="0.001" />
       <inertia
         ixx="0.00091529"
@@ -291,5 +291,5 @@
         rpy="0 0 0" />
       <mass
-        value="1.9415" />
+        value="0.001" />
       <inertia
         ixx="0.0015409"
@@ -349,5 +349,5 @@
         rpy="0 0 0" />
       <mass
-        value="0.049116" />
+        value="0.001" />
       <inertia
         ixx="6.9904E-08"
@@ -397,8 +397,16 @@
   <!-- ros_control plugin -->
   <gazebo>
+    <plugin name="gazebo_ros_control" filename="libgazebo_ros_control.so">
+      <robotNamespace>/sixrobot</robotNamespace>
+      <robotSimType>gazebo_ros_control/DefaultRobotHWSim</robotSimType>
+      <legacyModeNS>true</legacyModeNS>
+    </plugin>
+  </gazebo>
+  <!-- ros_control plugin -->
+  <!--<gazebo>
     <plugin name="ros_control" filename="lib_gazebo_ros_control.so">
-      <robotNamespace>/robot</robotNamespace>
+      <robotNamespace>/sixrobot</robotNamespace>
     </plugin>
-  </gazebo>
+  </gazebo>-->
   <!-- Gazebo-Specific Link Properties -->
   <gazebo reference="world_joint">
@@ -434,7 +442,26 @@
     <material>Gazebo/Blue</material>
   </gazebo>
+  <!-- Transmissions for ROS Control -->
+  <xacro:macro name="transmission_block" params="joint_name">
+    <transmission name="tran1">
+      <type>transmission_interface/SimpleTransmission</type>
+      <joint name="${joint_name}">
+        <hardwareInterface>hardware_interface/PositionJointInterface</hardwareInterface>
+      </joint>
+      <actuator name="motor1">
+        <hardwareInterface>hardware_interface/PositionJointInterface</hardwareInterface>
+        <mechanicalReduction>1</mechanicalReduction>
+      </actuator>
+    </transmission>
+  </xacro:macro>
+  <xacro:transmission_block joint_name="joint1"/>
+  <xacro:transmission_block joint_name="joint2"/>
+  <xacro:transmission_block joint_name="joint3"/>
+  <xacro:transmission_block joint_name="joint4"/>
+  <xacro:transmission_block joint_name="joint5"/>
+  <xacro:transmission_block joint_name="joint6"/>
   <!-- Transmissions -->
   <!-- Arm -->
-  <transmission name="tran1">
+  <!--<transmission name="tran1">
     <type>transmission_interface/SimpleTransmission</type>
     <joint name="joint1">
@@ -495,4 +522,4 @@
       <mechanicalReduction>1</mechanicalReduction>
     </actuator>
-  </transmission>
+  </transmission>-->
 </robot>
