Commit message: v2.0-gripper

File: src/sixrobot_description/urdf/dynamixel_arm_hardware.xacro (robot description, xacro)
@@ -1,4 +1,4 @@
 <?xml version="1.0"?>
-<robot name="arm_hardware" xmlns:xacro="http://ros.org/wiki/xacro">
+<robot name="arm_hardware" xmlns:xacro="http://www.ros.org/wiki/xacro">
   <xacro:property name="PI" value="3.14159"/>
   <xacro:property name="DYNAMIXEL_MESH_SCALE" value="0.001"/>

File: src/sixrobot_description/urdf/sensors/camera.urdf.xacro (robot description, xacro)
@@ -5,5 +5,5 @@
 <robot name="camera" xmlns:xacro="http://www.ros.org/wiki/xacro">
    <joint name="camera_joint" type="fixed">
-        <origin xyz="0.3 0 0.7" rpy="0 ${M_PI/2} 0"/>
+        <origin xyz="0 -0.5 0.7" rpy="0 ${M_PI/2} ${M_PI/2}"/>
         <parent link="base_link"/>
         <child link="camera_link"/>
@@ -23,4 +23,6 @@
            </geometry>
            <material name="red"/>
+           <color
+          rgba="255 0 0 1" />
        </visual>
        <inertial>
