Commit message: v2.0-gripper

File: src/sixrobot_description/urdf/sixrobot_anno_with_gripper.xacro (robot description, xacro)
@@ -366,4 +366,37 @@
    <!-- Attach the right gripper -->
    <gripper parent="tool0" color="Green" xyz="0 -0.015 0.01" rpy="0 0 ${M_PI}"/>
+  <!-- Gazebo-Specific Link Properties -->
+  <gazebo reference="world">
+    <selfCollide>true</selfCollide>
+    <material>Gazebo/White</material>
+  </gazebo>
+  <gazebo reference="base_link">
+    <selfCollide>true</selfCollide>
+    <material>Gazebo/White</material>
+  </gazebo>
+  <gazebo reference="Link1">
+    <implicitSpringDamper>1</implicitSpringDamper>
+    <material>Gazebo/Red</material>
+  </gazebo>
+  <gazebo reference="Link2">
+    <implicitSpringDamper>1</implicitSpringDamper>
+    <material>Gazebo/Green</material>
+  </gazebo>
+  <gazebo reference="Link3">
+    <implicitSpringDamper>1</implicitSpringDamper>
+    <material>Gazebo/Blue</material>
+  </gazebo>
+  <gazebo reference="Link4">
+    <implicitSpringDamper>1</implicitSpringDamper>
+    <material>Gazebo/Red</material>
+  </gazebo>
+  <gazebo reference="Link5">
+    <implicitSpringDamper>1</implicitSpringDamper>
+    <material>Gazebo/Green</material>
+  </gazebo>
+  <gazebo reference="Link6">
+    <implicitSpringDamper>1</implicitSpringDamper>
+    <material>Gazebo/Blue</material>
+  </gazebo>
   <!-- Transmissions for ROS Control -->
   <xacro:macro name="transmission_block" params="joint_name">
